File: Cap/capStone/capStone.kicad_pcb (KiCad board)
At the start: 2 copper layers, 24 x 16 mm, 77 parts, among them J1 USB_C_Receptacle_USB2.0_16P, J2 Micro_SD_Card_Det1, J4 Conn_01x10_Pin, SW1 BOOT, SW2 Reset, U1 ESP32-S3, U2 SX1262IMLTRT, U3 MAX-M10S, U4 LM1117MP-3.3V, U5 W25Q128JVS, U6 USBLC6-4SC6, Y1 32MHz, Y2 32MHz

Commit message: uploaded the 4 layer board
Parts:
- removed C14: 0.1uF, Capacitor_SMD:C_0402_1005Metric
- removed C15, C18, C20: 1uF, Capacitor_SMD:C_0402_1005Metric
- removed C19, C21: 100nF, Capacitor_SMD:C_0402_1005Metric
- removed C26: 10nF, Capacitor_SMD:C_0402_1005Metric
- removed J2: Micro_SD_Card_Det1, Connector_Card:SD_Card_Device_16mm_SlotDepth
- removed L2: 27nH, Inductor_SMD:L_0402_1005Metric
- removed R11, R7: 10k, Resistor_SMD:R_0402_1005Metric
- removed R22: 10Ohm, Resistor_SMD:R_0402_1005Metric
- removed R5, R6: 10kOhm, Resistor_SMD:R_0402_1005Metric
- removed U3: MAX-M10S, RF_GPS:ublox_MAX
- D3, D5: value LED_Small -> Green; footprint Resistor_SMD:R_0402_1005Metric -> LED_SMD:LED_0805_2012Metric
- D6: value LED_Small -> RED; footprint Resistor_SMD:R_0402_1005Metric -> LED_SMD:LED_0805_2012Metric
- R1, R2: value 5.1k -> 5.1k Ohm
- R23: value 1k -> 1k Ohm
- Y2: value 32MHz -> 40MHz
- moved C22 111.4 mm to (209.2, 31.1), turned to 90 degrees
- moved C23 111.2 mm to (209.2, 33.4), turned to 90 degrees
- moved U4 104.1 mm to (204.7, 33.9), turned to 180 degrees
- moved C13 103.0 mm to (208.9, 48.7)
- moved C12 102.6 mm to (208.9, 47.7)
- moved C16 99.9 mm to (191.8, 35.4), turned to 180 degrees
- moved J4 99.2 mm to (170.7, 46.1), turned to -90 degrees
- moved C11 98.6 mm to (199.2, 37.0)
- moved C7 96.7 mm to (195.1, 46.5), turned to 180 degrees
- moved C4 93.1 mm to (190.3, 40.2), turned to -90 degrees
- moved C2 92.8 mm to (191.3, 38.2), turned to -90 degrees
- moved C17 92.3 mm to (196.8, 36.5), turned to 45 degrees
- moved C6 91.5 mm to (185.4, 40.2), turned to -90 degrees
- moved R17 91.5 mm to (201.8, 41.4), turned to 180 degrees
- moved C8 91.4 mm to (191.7, 53.0), turned to 90 degrees
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Connections:
- C17 pad 1: /X_out -> /X_out_1
- C22 pad 1: VDD -> +5
- C41 pad 1: /USB_+5V -> +5
- D4 pad 4: VDD -> +5
- R9 pad 2: /X_in -> /X_in_1
- U1 pad 53: /X_out -> /X_out_1
- U1 pad 54: /X_in -> /X_in_1
- U4 pad 3: VDD -> +5
- U6 pad 5: /USB_+5V -> +5
- Y2 pad 3: /X_out -> /X_out_1
Routing:
- net +5: track 0.00 -> 75.9 mm, vias 0 -> 4
- net VDD_CPU: track 0.00 -> 60.3 mm, vias 0 -> 17
- net /GPIO35: track 0.00 -> 51.3 mm, vias 0 -> 1
- net /GPIO37: track 0.00 -> 49.0 mm, vias 0 -> 1
- net /GPIO34: track 0.00 -> 48.8 mm, vias 0 -> 1
- net /GPIO36: track 0.00 -> 47.7 mm, vias 0 -> 1
- net GND: track 0.00 -> 47.6 mm, vias 0 -> 51
- net /GPIO33: track 0.00 -> 44.8 mm, vias 0 -> 1
- net /VIN: track 0.00 -> 36.1 mm, vias 0 -> 1
- net /D_1_C-: track 0.00 -> 32.2 mm, vias 0 -> 2
- net /D_1_C+: track 0.00 -> 31.8 mm, vias 0 -> 2
- net Net-(D2-A2): track 0.00 -> 25.1 mm, vias 0 -> 3
- net Net-(D1-A2): track 0.00 -> 24.4 mm, vias 0 -> 2
- net /MISO: track 0.00 -> 21.9 mm, vias 0 -> 2
- net /RESET: track 0.00 -> 21.9 mm, vias 0 -> 2
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- added copper zone on In1.Cu, net GND
- added copper zone on In2.Cu, net VDD_CPU
Other:
- board size 24 x 16 mm -> 40 x 32 mm
- copper layers 2 -> 4
- board text added: "ESD3.3"
