File: Cap/capStone/capStone.kicad_sch (KiCad schematic)
At the start: 78 parts, among them J1 USB_C_Receptacle_USB2.0_16P, J2 Micro_SD_Card_Det1, J3 Conn_Coaxial, J4 Conn_01x10_Pin, SW1 BOOT, SW2 Reset, U1 ESP32-S3, U2 SX1262IMLTRT, U3 MAX-M10S, U4 LM1117MP-3.3V, U5 W25Q128JVS, U6 USBLC6-4SC6, Y1 32MHz, Y2 32MHz

Commit message: uploaded the 4 layer board
Parts:
- removed C14: 0.1uF, Capacitor_SMD:C_0402_1005Metric, symbol Device:C_Small
- removed C15: 1uF, Capacitor_SMD:C_0402_1005Metric, symbol Device:C_Small
- removed J2: Micro_SD_Card_Det1, Connector_Card:SD_Card_Device_16mm_SlotDepth, symbol Connector:Micro_SD_Card_Det1
- removed R5, R6: 10kOhm, Resistor_SMD:R_0402_1005Metric, symbol Device:R_Small
- added J5: Conn_02x02_Odd_Even, Library:4 way, symbol Connector_Generic:Conn_02x02_Odd_Even
- D3, D5, D6: footprint Resistor_SMD:R_0402_1005Metric -> LED_SMD:LED_0805_2012Metric
- Y2: value 32MHz -> 40MHz
Connections:
- net D_1_C+: now also J5.2 (Pin_2)
- net D_1_C-: now also J5.1 (Pin_1)
- net USB_+5V: no longer C41.1, U6.5 (VBUS)
- net X_in: no longer R9.2, U1.54 (XTAL_P)
- net X_out: no longer C17.1, U1.53 (XTAL_N), Y2.3
- net VDD renamed +5
- net +5: now also C41.1, U6.5 (VBUS)
- new net X_in_1: R9.2, U1.54 (XTAL_P)
- new net X_out_1: C17.1, U1.53 (XTAL_N), Y2.3
- no-connect marks 5 -> 3
Other:
- moved on the sheet: D3, D5, D6, D67, J4, R14, R15, R21, R23
